Commit message: Updated env, pybullet visualizor and robot_arm.urdf

File: 4-dof_rl_project/urdf/robot_arm.urdf (robot description, URDF)
Before this commit: robot snam1500_arm, 4 links, 3 joints
Links:
- removed link shoulder_link
- added link rotating_base_link; visual box size=0.05 0.004 0.052; visual box size=0.05 0.004 0.052
- link base_link: geometry visual box size=0.07 0.07 0.028
- link forearm_link: geometry visual cylinder length=0.11 radius=0.007; visual sphere radius=0.010
- link upper_arm_link: geometry visual box size=0.02 0.03 0.02; visual cylinder length=0.10 radius=0.008
Joints:
- joint joint_base: child shoulder_link -> rotating_base_link; origin xyz=0 0 0.08 -> xyz=0 0 0.028
- joint joint_shoulder: origin xyz=0.10 0 0 -> xyz=0 0 0.052; parent shoulder_link -> rotating_base_link
